Commit message: retracted code

File: rx1_description/urdf/rx1.urdf (robot description, URDF)
Before this commit: robot rx1, 24 links, 22 joints
Links:
- added link camera_link, mass 0.05; collision box size=0.01 0.01 0.01; visual box size=0.01 0.01 0.01
- added link head_depth_cam_mount_link, mass 0.05; collision mesh filename=package://rx1_description/meshes/head/head_depth_cam_mount_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; visual mesh filename=package://rx1_description/meshes/head/head_depth_cam_mount_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
- added link left_ear_link, mass 0.05; collision mesh filename=package://rx1_description/meshes/head/left_ear_link.stl; visual mesh filename=package://rx1_description/meshes/head/left_ear_link.stl
- added link neck_pitch_link, mass 0.05; collision mesh filename=package://rx1_description/meshes/head/neck_pitch_link.stl; visual mesh filename=package://rx1_description/meshes/head/neck_pitch_link.stl
- added link neck_yaw_link, mass 0.05; collision mesh filename=package://rx1_description/meshes/head/neck_yaw_link.stl; visual mesh filename=package://rx1_description/meshes/head/neck_yaw_link.stl
- added link right_ear_link, mass 0.05; collision mesh filename=package://rx1_description/meshes/head/right_ear_link.stl; visual mesh filename=package://rx1_description/meshes/head/right_ear_link.stl
- added link torso_link, mass 1.0; collision mesh filename=package://rx1_description/meshes/torso_link.stl; visual mesh filename=package://rx1_description/meshes/torso_link.stl
- added link torso_pitch_link, mass 0.5; collision cylinder length=0.03 radius=0.01; visual cylinder length=0.03 radius=0.015
- added link torso_roll_link, mass 0.5; collision cylinder length=0.03 radius=0.01; visual cylinder length=0.03 radius=0.015
- added link torso_yaw_link, mass 5.0; collision mesh filename=package://rx1_description/meshes/torso_yaw_link.stl; visual mesh filename=package://rx1_description/meshes/torso_yaw_link.stl
Joints:
- added joint base2torso_yaw_joint: type revolute, parent base_link, child torso_yaw_link, origin xyz=0.0 0.0 0.5825 rpy=0.0 0.0 0.0, axis 0.0 0.0 1.0, limit lower=-1.57075 upper=1.57075 effort=50.0 velocity=15.0
- added joint head_base2neck_yaw_joint: type revolute, parent head_base_link, child neck_yaw_link, origin xyz=0.0 0.0 0.0 rpy=0.0 0.0 0.0, axis 0.0 0.0 1.0, limit lower=-1.57075 upper=1.57075 effort=50.0 velocity=15.0
- added joint head_depth_cam_mount2camera_joint: type fixed, parent head_depth_cam_mount_link, child camera_link, origin xyz=0.05 0.0 0.03 rpy=0.0 0.0 0.0
- added joint head_depth_cam_mount2left_ear_joint: type revolute, parent head_depth_cam_mount_link, child left_ear_link, origin xyz=0.0 0.065 0.045 rpy=0.0 0.0 0.0, axis 0.0 1.0 0.0, limit lower=-1.57075 upper=1.57075 effort=50.0 velocity=15.0
- added joint head_depth_cam_mount2right_ear_joint: type revolute, parent head_depth_cam_mount_link, child right_ear_link, origin xyz=0.0 -0.065 0.045 rpy=0.0 0.0 0.0, axis 0.0 1.0 0.0, limit lower=-1.57075 upper=1.57075 effort=50.0 velocity=15.0
- added joint neck_pitch2head_depth_cam_mount_joint: type revolute, parent neck_pitch_link, child head_depth_cam_mount_link, origin xyz=-0.01 0.0 0.1 rpy=0.0 0.0 0.0, axis 1.0 0.0 0.0, limit lower=-1.57075 upper=1.57075 effort=50.0 velocity=15.0
- added joint neck_yaw2pitch_joint: type revolute, parent neck_yaw_link, child neck_pitch_link, origin xyz=0.0 0.0 0.035 rpy=0.0 0.0 0.0, axis 0.0 1.0 0.0, limit lower=-1.57075 upper=1.57075 effort=50.0 velocity=15.0
- added joint torso2head_base_joint: type fixed, parent torso_link, child head_base_link, origin xyz=0.0 0.0 0.21 rpy=0.0 0.0 0.0
- added joint torso_pitch2roll_joint: type revolute, parent torso_pitch_link, child torso_roll_link, origin xyz=0.0 0.0 0.0 rpy=0.0 0.0 0.0, axis 1.0 0.0 0.0, limit lower=-0.785375 upper=0.785375 effort=50.0 velocity=15.0
- added joint torso_roll2torso_joint: type fixed, parent torso_roll_link, child torso_link, origin xyz=0.0 0.0 0.08 rpy=0.0 0.0 0.0
- added joint torso_yaw2pitch_joint: type revolute, parent torso_yaw_link, child torso_pitch_link, origin xyz=0.0 0.0 0.15 rpy=0.0 0.0 0.0, axis 0.0 1.0 0.0, limit lower=-0.785375 upper=0.785375 effort=50.0 velocity=15.0

File: rx1_description/urdf/rx1.urdf.xacro (robot description, xacro)
@@ -37,4 +37,113 @@
         </collision>
     </link>
+    <!--                            TORSO START                         -->
+    <link name="torso_yaw_link">
+        <inertial>
+            <mass value="5.0" />
+            <inertia ixx="1.0" ixy="0.0" ixz="0.0" iyy="1.0" iyz="0.0" izz="1.0" />
+        </inertial>
+        <visual>
+            <geometry>
+                <mesh filename="package://rx1_description/meshes/torso_yaw_link.stl"/>
+            </geometry>
+            <origin rpy="0 0 0" xyz="0 0 0"/>
+            <material name="white"/>
+        </visual>
+        <collision>
+            <geometry>
+                <mesh filename="package://rx1_description/meshes/torso_yaw_link.stl"/>
+            </geometry>
+            <origin rpy="0 0 0" xyz="0 0 0"/>
+        </collision>
+    </link>
+    <joint name="base2torso_yaw_joint" type="revolute">
+        <axis xyz="0 0 1" />
+        <limit effort="${motor_torque}" lower="${-0.5*pi}" upper="${0.5*pi}" velocity="${motor_vec}"/>
+        <dynamics damping="0.5" friction="5.0" />
+        <origin xyz="0 0 0.5825" rpy="0 0 0" />
+        <parent link="base_link" />
+        <child link="torso_yaw_link" />
+    </joint>
+    <link name="torso_pitch_link">
+        <inertial>
+            <mass value="0.5" />
+            <inertia ixx="1.0" ixy="0.0" ixz="0.0" iyy="1.0" iyz="0.0" izz="1.0" />
+        </inertial>
+        <visual>
+            <geometry>
+                <cylinder length="0.03" radius="0.015" />
+            </geometry>
+            <origin rpy="${0.5*pi} 0 0" xyz="0 0 0"/>
+            <material name="blue"/>
+        </visual>
+        <collision>
+            <geometry>
+                <cylinder length="0.03" radius="0.01" />
+            </geometry>
+            <origin rpy="${0.5*pi} 0 0" xyz="0 0 0"/>
+        </collision>
+    </link>
+    <joint name="torso_yaw2pitch_joint" type="revolute">
+        <axis xyz="0 1 0" />
+        <limit effort="${motor_torque}" lower="${-0.25*pi}" upper="${0.25*pi}" velocity="${motor_vec}"/>
+        <dynamics damping="0.5" friction="0.1" />
+        <origin xyz="0 0 0.15" rpy="0 0 0" />
+        <parent link="torso_yaw_link" />
+        <child link="torso_pitch_link" />
+    </joint>
+    <link name="torso_roll_link">
+        <inertial>
+            <mass value="0.5" />
+            <inertia ixx="1.0" ixy="0.0" ixz="0.0" iyy="1.0" iyz="0.0" izz="1.0" />
+        </inertial>
+        <visual>
+            <geometry>
+                <cylinder length="0.03" radius="0.015" />
+            </geometry>
+            <origin rpy="0 ${0.5*pi} 0" xyz="0 0 0"/>
+            <material name="red"/>
+        </visual>
+        <collision>
+            <geometry>
+                <cylinder length="0.03" radius="0.01" />
+            </geometry>
+            <origin rpy="0 ${0.5*pi} 0" xyz="0 0 0"/>
+        </collision>
+    </link>
+    <joint name="torso_pitch2roll_joint" type="revolute">
+        <axis xyz="1 0 0" />
+        <limit effort="${motor_torque}" lower="${-0.25*pi}" upper="${0.25*pi}" velocity="${motor_vec}"/>
+        <dynamics damping="0.5" friction="0.1" />
+        <origin xyz="0 0 0" rpy="0 0 0" />
+        <parent link="torso_pitch_link" />
+        <child link="torso_roll_link" />
+    </joint>
+    <link name="torso_link">
+        <inertial>
+            <mass value="1" />
+            <inertia ixx="4.16666667e-06" ixy="0.0" ixz="0.0" iyy="6.6666666667e-6" iyz="0.0" izz="04.16666667e-06" />
+        </inertial>
+        <visual>
+            <geometry>
+                <!--box size="0.03 0.12 0.02" /-->
+                <mesh filename="package://rx1_description/meshes/torso_link.stl"/>
+            </geometry>
+            <origin rpy="0 0 0" xyz="0 0 0"/>
+            <material name="white"/>
+        </visual>
+        <collision>
+            <geometry>
+                <!--box size="0.03 0.12 0.02" /-->
+                <mesh filename="package://rx1_description/meshes/torso_link.stl"/>
+            </geometry>
+            <origin rpy="0 0 0" xyz="0 0 0"/>
+        </collision>
+    </link>
+    <joint name="torso_roll2torso_joint" type="fixed">
+        <origin xyz="0 0 0.08" rpy="0 0 0" />
+        <parent link="torso_roll_link" />
+        <child link="torso_link" />
+    </joint>
+    <!--                            TORSO END                         -->
     <!--                            HEAD START                        -->
     <link name="head_base_link">
@@ -57,4 +166,168 @@
         </collision>
     </link>
+    <joint name="torso2head_base_joint" type="fixed">
+        <origin xyz="0 0 0.21" rpy="0 0 0" />
+        <parent link="torso_link" />
+        <child link="head_base_link" />
+    </joint>
+    <link name="neck_yaw_link">
+        <inertial>
+            <mass value="0.05" />
+            <inertia ixx="4.16666667e-06" ixy="0.0" ixz="0.0" iyy="6.6666666667e-6" iyz="0.0" izz="04.16666667e-06" />
+        </inertial>
+        <visual>
+            <geometry>
+                <mesh filename="package://rx1_description/meshes/head/neck_yaw_link.stl"/>
+            </geometry>
+            <origin rpy="0 0 0" xyz="0 0 0"/>
+            <material name="white"/>
+        </visual>
+        <collision>
+            <geometry>
+                <mesh filename="package://rx1_description/meshes/head/neck_yaw_link.stl"/>
+            </geometry>
+            <origin rpy="0 0 0" xyz="0 0 0"/>
+        </collision>
+    </link>
+    <joint name="head_base2neck_yaw_joint" type="revolute">
+        <axis xyz="0 0 1" />
+        <limit effort="${motor_torque}" lower="${-0.5*pi}" upper="${0.5*pi}" velocity="${motor_vec}"/>
+        <dynamics damping="0.5" friction="0.1" />
+        <origin xyz="0 0 0" rpy="0 0 0" />
+        <parent link="head_base_link" />
+        <child link="neck_yaw_link" />
+    </joint>
+    <link name="neck_pitch_link">
+        <inertial>
+            <mass value="0.05" />
+            <inertia ixx="4.16666667e-06" ixy="0.0" ixz="0.0" iyy="6.6666666667e-6" iyz="0.0" izz="04.16666667e-06" />
+        </inertial>
+        <visual>
+            <geometry>
+                <mesh filename="package://rx1_description/meshes/head/neck_pitch_link.stl"/>
+            </geometry>
+            <origin rpy="0 0 0" xyz="0 0 0"/>
+            <material name="white"/>
+        </visual>
+        <collision>
+            <geometry>
+                <mesh filename="package://rx1_description/meshes/head/neck_pitch_link.stl"/>
+            </geometry>
+            <origin rpy="0 0 0" xyz="0 0 0"/>
+        </collision>
+    </link>
+    <joint name="neck_yaw2pitch_joint" type="revolute">
+        <axis xyz="0 1 0" />
+        <limit effort="${motor_torque}" lower="${-0.5*pi}" upper="${0.5*pi}" velocity="${motor_vec}"/>
+        <dynamics damping="0.5" friction="0.1" />
+        <origin xyz="0 0 0.035" rpy="0 0 0" />
+        <parent link="neck_yaw_link" />
+        <child link="neck_pitch_link" />
+    </joint>
+    <link name="head_depth_cam_mount_link">
+        <inertial>
+            <mass value="0.05" />
+            <inertia ixx="4.16666667e-06" ixy="0.0" ixz="0.0" iyy="6.6666666667e-6" iyz="0.0" izz="04.16666667e-06" />
+        </inertial>
+        <visual>
+            <geometry>
+                <mesh filename="package://rx1_description/meshes/head/head_depth_cam_mount_link.stl"/>
+            </geometry>
+            <origin rpy="0 0 0" xyz="0 0 0"/>
+            <material name="white"/>
+        </visual>
+        <collision>
+            <geometry>
+                <mesh filename="package://rx1_description/meshes/head/head_depth_cam_mount_link.stl"/>
+            </geometry>
+            <origin rpy="0 0 0" xyz="0 0 0"/>
+        </collision>
+    </link>
+    <joint name="neck_pitch2head_depth_cam_mount_joint" type="revolute">
+        <axis xyz="1 0 0" />
+        <limit effort="${motor_torque}" lower="${-0.5*pi}" upper="${0.5*pi}" velocity="${motor_vec}"/>
+        <dynamics damping="0.1" friction="0.0" />
+        <origin xyz="-0.01 0 0.1" rpy="0 0 0" />
+        <parent link="neck_pitch_link" />
+        <child link="head_depth_cam_mount_link" />
+    </joint>
+    <link name="camera_link">
+        <inertial>
+            <mass value="0.05" />
+            <inertia ixx="4.16666667e-06" ixy="0.0" ixz="0.0" iyy="6.6666666667e-6" iyz="0.0" izz="04.16666667e-06" />
+        </inertial>
+        <visual>
+            <geometry>
+                <box size="0.01 0.01 0.01" />
+            </geometry>
+            <origin rpy="0 0 0" xyz="0 0 0"/>
+            <material name="white"/>
+        </visual>
+        <collision>
+            <geometry>
+                <box size="0.01 0.01 0.01" />
+            </geometry>
+            <origin rpy="0 0 0" xyz="0 0 0"/>
+        </collision>
+    </link>
+    <joint name="head_depth_cam_mount2camera_joint" type="fixed">
+        <origin xyz="0.05 0 0.03" rpy="0 0 0" />
+        <parent link="head_depth_cam_mount_link" />
+        <child link="camera_link" />
+    </joint>
+    <link name="right_ear_link">
+        <inertial>
+            <mass value="0.05" />
+            <inertia ixx="4.16666667e-06" ixy="0.0" ixz="0.0" iyy="6.6666666667e-6" iyz="0.0" izz="04.16666667e-06" />
+        </inertial>
+        <visual>
+            <geometry>
+                <mesh filename="package://rx1_description/meshes/head/right_ear_link.stl"/>
+            </geometry>
+            <origin rpy="0 0 0" xyz="0 0 0"/>
+            <material name="white"/>
+        </visual>
+        <collision>
+            <geometry>
+                <mesh filename="package://rx1_description/meshes/head/right_ear_link.stl"/>
+            </geometry>
+            <origin rpy="0 0 0" xyz="0 0 0"/>
+        </collision>
+    </link>
+    <joint name="head_depth_cam_mount2right_ear_joint" type="revolute">
+        <axis xyz="0 1 0" />
+        <limit effort="${motor_torque}" lower="${-0.5*pi}" upper="${0.5*pi}" velocity="${motor_vec}"/>
+        <dynamics damping="0.1" friction="0.0" />
+        <origin xyz="0 -0.065 0.045" rpy="0 0 0" />
+        <parent link="head_depth_cam_mount_link" />
+        <child link="right_ear_link" />
+    </joint>
+    <link name="left_ear_link">
+        <inertial>
+            <mass value="0.05" />
+            <inertia ixx="4.16666667e-06" ixy="0.0" ixz="0.0" iyy="6.6666666667e-6" iyz="0.0" izz="04.16666667e-06" />
+        </inertial>
+        <visual>
+            <geometry>
+                <mesh filename="package://rx1_description/meshes/head/left_ear_link.stl"/>
+            </geometry>
+            <origin rpy="0 0 0" xyz="0 0 0"/>
+            <material name="white"/>
+        </visual>
+        <collision>
+            <geometry>
+                <mesh filename="package://rx1_description/meshes/head/left_ear_link.stl"/>
+            </geometry>
+            <origin rpy="0 0 0" xyz="0 0 0"/>
+        </collision>
+    </link>
+    <joint name="head_depth_cam_mount2left_ear_joint" type="revolute">
+        <axis xyz="0 1 0" />
+        <limit effort="${motor_torque}" lower="${-0.5*pi}" upper="${0.5*pi}" velocity="${motor_vec}"/>
+        <dynamics damping="0.1" friction="0.0" />
+        <origin xyz="0 0.065 0.045" rpy="0 0 0" />
+        <parent link="head_depth_cam_mount_link" />
+        <child link="left_ear_link" />
+    </joint>
     <!--                            HEAD END                           -->
     <!--                            ARM START                          -->
