Commit message: code

File: rx1_description/urdf/rx1.urdf (robot description, URDF)
Before this commit: robot rx1, 34 links, 33 joints
Links:
- removed link camera_link
- removed link head_depth_cam_mount_link
- removed link left_ear_link
- removed link neck_pitch_link
- removed link neck_yaw_link
- removed link right_ear_link
Joints:
- removed joint head_base2neck_yaw_joint
- removed joint head_depth_cam_mount2camera_joint
- removed joint head_depth_cam_mount2left_ear_joint
- removed joint head_depth_cam_mount2right_ear_joint
- removed joint neck_pitch2head_depth_cam_mount_joint
- removed joint neck_yaw2pitch_joint

File: rx1_description/urdf/rx1.urdf.xacro (robot description, xacro)
@@ -166,168 +166,4 @@
         </collision>
     </link>
-    <joint name="torso2head_base_joint" type="fixed">
-        <origin xyz="0 0 0.21" rpy="0 0 0" />
-        <parent link="torso_link" />
-        <child link="head_base_link" />
-    </joint>
-    <link name="neck_yaw_link">
-        <inertial>
-            <mass value="0.05" />
-            <inertia ixx="4.16666667e-06" ixy="0.0" ixz="0.0" iyy="6.6666666667e-6" iyz="0.0" izz="04.16666667e-06" />
-        </inertial>
-        <visual>
-            <geometry>
-                <mesh filename="package://rx1_description/meshes/head/neck_yaw_link.stl"/>
-            </geometry>
-            <origin rpy="0 0 0" xyz="0 0 0"/>
-            <material name="white"/>
-        </visual>
-        <collision>
-            <geometry>
-                <mesh filename="package://rx1_description/meshes/head/neck_yaw_link.stl"/>
-            </geometry>
-            <origin rpy="0 0 0" xyz="0 0 0"/>
-        </collision>
-    </link>
-    <joint name="head_base2neck_yaw_joint" type="revolute">
-        <axis xyz="0 0 1" />
-        <limit effort="${motor_torque}" lower="${-0.5*pi}" upper="${0.5*pi}" velocity="${motor_vec}"/>
-        <dynamics damping="0.5" friction="0.1" />
-        <origin xyz="0 0 0" rpy="0 0 0" />
-        <parent link="head_base_link" />
-        <child link="neck_yaw_link" />
-    </joint>
-    <link name="neck_pitch_link">
-        <inertial>
-            <mass value="0.05" />
-            <inertia ixx="4.16666667e-06" ixy="0.0" ixz="0.0" iyy="6.6666666667e-6" iyz="0.0" izz="04.16666667e-06" />
-        </inertial>
-        <visual>
-            <geometry>
-                <mesh filename="package://rx1_description/meshes/head/neck_pitch_link.stl"/>
-            </geometry>
-            <origin rpy="0 0 0" xyz="0 0 0"/>
-            <material name="white"/>
-        </visual>
-        <collision>
-            <geometry>
-                <mesh filename="package://rx1_description/meshes/head/neck_pitch_link.stl"/>
-            </geometry>
-            <origin rpy="0 0 0" xyz="0 0 0"/>
-        </collision>
-    </link>
-    <joint name="neck_yaw2pitch_joint" type="revolute">
-        <axis xyz="0 1 0" />
-        <limit effort="${motor_torque}" lower="${-0.5*pi}" upper="${0.5*pi}" velocity="${motor_vec}"/>
-        <dynamics damping="0.5" friction="0.1" />
-        <origin xyz="0 0 0.035" rpy="0 0 0" />
-        <parent link="neck_yaw_link" />
-        <child link="neck_pitch_link" />
-    </joint>
-    <link name="head_depth_cam_mount_link">
-        <inertial>
-            <mass value="0.05" />
-            <inertia ixx="4.16666667e-06" ixy="0.0" ixz="0.0" iyy="6.6666666667e-6" iyz="0.0" izz="04.16666667e-06" />
-        </inertial>
-        <visual>
-            <geometry>
-                <mesh filename="package://rx1_description/meshes/head/head_depth_cam_mount_link.stl"/>
-            </geometry>
-            <origin rpy="0 0 0" xyz="0 0 0"/>
-            <material name="white"/>
-        </visual>
-        <collision>
-            <geometry>
-                <mesh filename="package://rx1_description/meshes/head/head_depth_cam_mount_link.stl"/>
-            </geometry>
-            <origin rpy="0 0 0" xyz="0 0 0"/>
-        </collision>
-    </link>
-    <joint name="neck_pitch2head_depth_cam_mount_joint" type="revolute">
-        <axis xyz="1 0 0" />
-        <limit effort="${motor_torque}" lower="${-0.5*pi}" upper="${0.5*pi}" velocity="${motor_vec}"/>
-        <dynamics damping="0.1" friction="0.0" />
-        <origin xyz="-0.01 0 0.1" rpy="0 0 0" />
-        <parent link="neck_pitch_link" />
-        <child link="head_depth_cam_mount_link" />
-    </joint>
-    <link name="camera_link">
-        <inertial>
-            <mass value="0.05" />
-            <inertia ixx="4.16666667e-06" ixy="0.0" ixz="0.0" iyy="6.6666666667e-6" iyz="0.0" izz="04.16666667e-06" />
-        </inertial>
-        <visual>
-            <geometry>
-                <box size="0.01 0.01 0.01" />
-            </geometry>
-            <origin rpy="0 0 0" xyz="0 0 0"/>
-            <material name="white"/>
-        </visual>
-        <collision>
-            <geometry>
-                <box size="0.01 0.01 0.01" />
-            </geometry>
-            <origin rpy="0 0 0" xyz="0 0 0"/>
-        </collision>
-    </link>
-    <joint name="head_depth_cam_mount2camera_joint" type="fixed">
-        <origin xyz="0.05 0 0.03" rpy="0 0 0" />
-        <parent link="head_depth_cam_mount_link" />
-        <child link="camera_link" />
-    </joint>
-    <link name="right_ear_link">
-        <inertial>
-            <mass value="0.05" />
-            <inertia ixx="4.16666667e-06" ixy="0.0" ixz="0.0" iyy="6.6666666667e-6" iyz="0.0" izz="04.16666667e-06" />
-        </inertial>
-        <visual>
-            <geometry>
-                <mesh filename="package://rx1_description/meshes/head/right_ear_link.stl"/>
-            </geometry>
-            <origin rpy="0 0 0" xyz="0 0 0"/>
-            <material name="white"/>
-        </visual>
-        <collision>
-            <geometry>
-                <mesh filename="package://rx1_description/meshes/head/right_ear_link.stl"/>
-            </geometry>
-            <origin rpy="0 0 0" xyz="0 0 0"/>
-        </collision>
-    </link>
-    <joint name="head_depth_cam_mount2right_ear_joint" type="revolute">
-        <axis xyz="0 1 0" />
-        <limit effort="${motor_torque}" lower="${-0.5*pi}" upper="${0.5*pi}" velocity="${motor_vec}"/>
-        <dynamics damping="0.1" friction="0.0" />
-        <origin xyz="0 -0.065 0.045" rpy="0 0 0" />
-        <parent link="head_depth_cam_mount_link" />
-        <child link="right_ear_link" />
-    </joint>
-    <link name="left_ear_link">
-        <inertial>
-            <mass value="0.05" />
-            <inertia ixx="4.16666667e-06" ixy="0.0" ixz="0.0" iyy="6.6666666667e-6" iyz="0.0" izz="04.16666667e-06" />
-        </inertial>
-        <visual>
-            <geometry>
-                <mesh filename="package://rx1_description/meshes/head/left_ear_link.stl"/>
-            </geometry>
-            <origin rpy="0 0 0" xyz="0 0 0"/>
-            <material name="white"/>
-        </visual>
-        <collision>
-            <geometry>
-                <mesh filename="package://rx1_description/meshes/head/left_ear_link.stl"/>
-            </geometry>
-            <origin rpy="0 0 0" xyz="0 0 0"/>
-        </collision>
-    </link>
-    <joint name="head_depth_cam_mount2left_ear_joint" type="revolute">
-        <axis xyz="0 1 0" />
-        <limit effort="${motor_torque}" lower="${-0.5*pi}" upper="${0.5*pi}" velocity="${motor_vec}"/>
-        <dynamics damping="0.1" friction="0.0" />
-        <origin xyz="0 0.065 0.045" rpy="0 0 0" />
-        <parent link="head_depth_cam_mount_link" />
-        <child link="left_ear_link" />
-    </joint>
     <!--                            HEAD END                           -->
     <!--                            ARM START                          -->

Commit message: Update rx1.urdf

File: rx1_description/urdf/rx1.urdf (robot description, URDF)
Before this commit: robot rx1, 28 links, 27 joints
Links:
- removed link torso_pitch_link
- removed link torso_roll_link
- removed link torso_yaw_link
Joints:
- removed joint base2torso_yaw_joint
- removed joint torso_pitch2roll_joint
- removed joint torso_roll2torso_joint
- removed joint torso_yaw2pitch_joint

Commit message: Update rx1.urdf

File: rx1_description/urdf/rx1.urdf (robot description, URDF)
Before this commit: robot rx1, 25 links, 23 joints
Links:
- added link torso_pitch_link, mass 0.5; collision cylinder length=0.03 radius=0.01; visual cylinder length=0.03 radius=0.015
- added link torso_roll_link, mass 0.5; collision cylinder length=0.03 radius=0.01; visual cylinder length=0.03 radius=0.015
- added link torso_yaw_link, mass 5.0; collision mesh filename=package://rx1_description/meshes/torso_yaw_link.stl; visual mesh filename=package://rx1_description/meshes/torso_yaw_link.stl
Joints:
- added joint base2torso_yaw_joint: type revolute, parent base_link, child torso_yaw_link, origin xyz=0.0 0.0 0.5825 rpy=0.0 0.0 0.0, axis 0.0 0.0 1.0, limit lower=-1.57075 upper=1.57075 effort=50.0 velocity=15.0
- added joint torso_pitch2roll_joint: type revolute, parent torso_pitch_link, child torso_roll_link, origin xyz=0.0 0.0 0.0 rpy=0.0 0.0 0.0, axis 1.0 0.0 0.0, limit lower=-0.785375 upper=0.785375 effort=50.0 velocity=15.0
- added joint torso_roll2torso_joint: type fixed, parent torso_roll_link, child torso_link, origin xyz=0.0 0.0 0.08 rpy=0.0 0.0 0.0
- added joint torso_yaw2pitch_joint: type revolute, parent torso_yaw_link, child torso_pitch_link, origin xyz=0.0 0.0 0.15 rpy=0.0 0.0 0.0, axis 0.0 1.0 0.0, limit lower=-0.785375 upper=0.785375 effort=50.0 velocity=15.0

Commit message: Update rx1.urdf

File: rx1_description/urdf/rx1.urdf (robot description, URDF)
Before this commit: robot rx1, 28 links, 27 joints
Links:
- removed link torso_link
- removed link torso_pitch_link
- removed link torso_roll_link
- removed link torso_yaw_link
Joints:
- removed joint base2torso_yaw_joint
- removed joint torso2head_base_joint
- removed joint torso_pitch2roll_joint
- removed joint torso_roll2torso_joint
- removed joint torso_yaw2pitch_joint
- added joint head_base2base_link: type fixed, parent head_base_link, child base_link, origin xyz=0.0 -0.12 -0.05 rpy=1.04706195 0.0 0.0

Commit message: Update rx1.urdf

File: rx1_description/urdf/rx1.urdf (robot description, URDF)
Before this commit: robot rx1, 24 links, 23 joints
Links:
- added link torso_link, mass 1.0; collision mesh filename=package://rx1_description/meshes/torso_link.stl; visual mesh filename=package://rx1_description/meshes/torso_link.stl
- added link torso_pitch_link, mass 0.5; collision cylinder length=0.03 radius=0.01; visual cylinder length=0.03 radius=0.015
- added link torso_roll_link, mass 0.5; collision cylinder length=0.03 radius=0.01; visual cylinder length=0.03 radius=0.015
- added link torso_yaw_link, mass 5.0; collision mesh filename=package://rx1_description/meshes/torso_yaw_link.stl; visual mesh filename=package://rx1_description/meshes/torso_yaw_link.stl
Joints:
- removed joint head_base2base_link
- added joint base2torso_yaw_joint: type revolute, parent base_link, child torso_yaw_link, origin xyz=0.0 0.0 0.5825 rpy=0.0 0.0 0.0, axis 0.0 0.0 1.0, limit lower=-1.57075 upper=1.57075 effort=50.0 velocity=15.0
- added joint torso2head_base_joint: type fixed, parent torso_link, child head_base_link, origin xyz=0.0 0.0 0.21 rpy=0.0 0.0 0.0
- added joint torso_pitch2roll_joint: type revolute, parent torso_pitch_link, child torso_roll_link, origin xyz=0.0 0.0 0.0 rpy=0.0 0.0 0.0, axis 1.0 0.0 0.0, limit lower=-0.785375 upper=0.785375 effort=50.0 velocity=15.0
- added joint torso_roll2torso_joint: type fixed, parent torso_roll_link, child torso_link, origin xyz=0.0 0.0 0.08 rpy=0.0 0.0 0.0
- added joint torso_yaw2pitch_joint: type revolute, parent torso_yaw_link, child torso_pitch_link, origin xyz=0.0 0.0 0.15 rpy=0.0 0.0 0.0, axis 0.0 1.0 0.0, limit lower=-0.785375 upper=0.785375 effort=50.0 velocity=15.0

Commit message: Update rx1.urdf

File: rx1_description/urdf/rx1.urdf (robot description, URDF)
Before this commit: robot rx1, 28 links, 27 joints
Links:
- removed link torso_link
- removed link torso_pitch_link
- removed link torso_roll_link
- removed link torso_yaw_link
Joints:
- removed joint base2torso_yaw_joint
- removed joint torso2head_base_joint
- removed joint torso_pitch2roll_joint
- removed joint torso_roll2torso_joint
- removed joint torso_yaw2pitch_joint
- added joint base2head_base: type fixed, parent base_link, child head_base, origin xyz=0.0 0.0 0.5825 rpy=0.0 0.0 0.0

Commit message: Update rx1.urdf

File: rx1_description/urdf/rx1.urdf (robot description, URDF)
Before this commit: robot rx1, 24 links, 23 joints
Joints:
- removed joint base2head_base
- added joint base2head_base_joint: type fixed, parent base_link, child head_base_link, origin xyz=0.0 0.0 0.7925 rpy=0.0 0.0 0.0
- joint left_shoul2shoul_rot_joint: limit lower=-0.5026400000000001 upper=1.57075 effort=50.0 velocity=15.0 -> lower=-0.50264 upper=1.57075 effort=50.0 velocity=15.0
- joint left_shoul_base2shoul_joint: limit lower=-2.5132000000000003 upper=2.5132000000000003 effort=50.0 velocity=15.0 -> lower=-2.5132 upper=2.5132 effort=50.0 velocity=15.0
- joint right_shoul2shoul_rot_joint: limit lower=-1.57075 upper=0.5026400000000001 effort=50.0 velocity=15.0 -> lower=-1.57075 upper=0.50264 effort=50.0 velocity=15.0
- joint right_shoul_base2shoul_joint: limit lower=-2.5132000000000003 upper=2.5132000000000003 effort=50.0 velocity=15.0 -> lower=-2.5132 upper=2.5132 effort=50.0 velocity=15.0

Commit message: Update rx1.urdf

File: rx1_description/urdf/rx1.urdf (robot description, URDF)
Before this commit: robot rx1, 24 links, 23 joints
Links:
- removed link head_base_link
- added link torso_link, mass 0.05; collision mesh filename=package://rx1_description/meshes/head/head_base_link.stl; visual mesh filename=package://rx1_description/meshes/head/head_base_link.stl
Joints:
- removed joint base2head_base_joint
- removed joint head_base2left_shoul_base_joint
- removed joint head_base2right_shoul_base_joint
- added joint base2torso_link_joint: type fixed, parent base_link, child torso_link, origin xyz=0.0 0.0 0.7925 rpy=0.0 0.0 0.0
- added joint torso_link2left_shoul_base_joint: type fixed, parent torso_link, child left_shoul_base_link, origin xyz=0.0 0.12 -0.05 rpy=-1.04706195 0.0 0.0
- added joint torso_link2right_shoul_base_joint: type fixed, parent torso_link, child right_shoul_base_link, origin xyz=0.0 -0.12 -0.05 rpy=1.04706195 0.0 0.0

Commit message: Update rx1.urdf

File: rx1_description/urdf/rx1.urdf (robot description, URDF)
Before this commit: robot rx1, 24 links, 23 joints
Links:
- link torso_link: geometry collision mesh filename=package://rx1_description/meshes/head/torso_link.stl; visual mesh filename=package://rx1_description/meshes/head/torso_link.stl

Commit message: Update rx1.urdf

File: rx1_description/urdf/rx1.urdf (robot description, URDF)
Before this commit: robot rx1, 24 links, 23 joints
Links:
- link torso_link: geometry collision mesh filename=package://rx1_description/meshes/torso_link.stl; visual mesh filename=package://rx1_description/meshes/torso_link.stl

Commit message: Update rx1.urdf

File: rx1_description/urdf/rx1.urdf (robot description, URDF)
Before this commit: robot rx1, 24 links, 23 joints
Links:
- removed link torso_link
- added link head_base_link, mass 0.05; collision mesh filename=package://rx1_description/meshes/head/head_base_link.stl; visual mesh filename=package://rx1_description/meshes/head/head_base_link.stl
Joints:
- removed joint base2torso_link_joint
- removed joint torso_link2left_shoul_base_joint
- removed joint torso_link2right_shoul_base_joint
- added joint base2head_base_joint: type fixed, parent base_link, child head_base_link, origin xyz=0.0 0.0 0.7925 rpy=0.0 0.0 0.0
- added joint head_base2left_shoul_base_joint: type fixed, parent head_base_link, child left_shoul_base_link, origin xyz=0.0 0.12 -0.05 rpy=-1.04706195 0.0 0.0
- added joint head_base2right_shoul_base_joint: type fixed, parent head_base_link, child right_shoul_base_link, origin xyz=0.0 -0.12 -0.05 rpy=1.04706195 0.0 0.0

Commit message: Update rx1.urdf

File: rx1_description/urdf/rx1.urdf (robot description, URDF)
Before this commit: robot rx1, 24 links, 23 joints
Links:
- added link torso_link, mass 1.0; collision mesh filename=package://rx1_description/meshes/torso_link.stl; visual mesh filename=package://rx1_description/meshes/torso_link.stl
Joints:
- removed joint base2head_base_joint
- added joint base2torso_joint: type fixed, parent base_link, child torso_link, origin xyz=0.0 0.0 0.5825 rpy=0.0 0.0 0.0
- added joint torso2head_base_joint: type fixed, parent torso_link, child head_base_link, origin xyz=0.0 0.0 0.21 rpy=0.0 0.0 0.0

Commit message: Update rx1.urdf

File: rx1_description/urdf/rx1.urdf (robot description, URDF)
Before this commit: robot rx1, 25 links, 24 joints
Joints:
- joint base2torso_joint: origin xyz=0.0 0.0 0.5825 rpy=0.0 0.0 0.0 -> xyz=0.0 0.0 0.1 rpy=0.0 0.0 0.0
- joint torso2head_base_joint: origin xyz=0.0 0.0 0.21 rpy=0.0 0.0 0.0 -> xyz=0.0 0.0 4.385 rpy=0.0 0.0 0.0

Commit message: Update rx1.urdf

File: rx1_description/urdf/rx1.urdf (robot description, URDF)
Before this commit: robot rx1, 25 links, 24 joints
Joints:
- joint base2torso_joint: origin xyz=0.0 0.0 0.1 rpy=0.0 0.0 0.0 -> xyz=0.0 0.0 0.5825 rpy=0.0 0.0 0.0
- joint torso2head_base_joint: origin xyz=0.0 0.0 4.385 rpy=0.0 0.0 0.0 -> xyz=0.0 0.0 0.21 rpy=0.0 0.0 0.0
